File: Hardware/FilPilote.sch (KiCad schematic (older format))
At the start: 33 parts, among them IC1 MOC3041M, IC2 MOC3041M, IC3 MOC3041M, IC4 MOC3041M, IC5 MOC3041M, IC6 MOC3041M, P1 CONN_01X03, P2 CONN_01X03, P3 CONN_01X07

Commit message: Remove useless earth connection
Connections:
- net Terre: no longer names the net of P1.1 (P1)
- no-connect marks 0 -> 1
Changed lines of the file:
@@
 Wire Wire Line
 	5150 1300 5150 1200
-Text GLabel 5100 1100 0    60   Input ~ 0
-Terre
-Wire Wire Line
-	5100 1100 5150 1100
+NoConn ~ 5150 1100
 $EndSCHEMATC

Commit message: Move to kicad 4.0.0 RC1
Parts:
- D1, D2, D3, D4, D5, D6: footprint Diodes_ThroughHole:Diode_DO-41_SOD81_Horizontal_RM10 -> Discret:D4
- IC1, IC2, IC3, IC4, IC5, IC6: symbol MOC3041M -> MOC3041M-RESCUE-FilPilote
- R1, R10, R11, R12, R2, R3, R4, R5, R6, R7, R8, R9: symbol R -> R-RESCUE-FilPilote
Connections:
- net GND: now also D10.1 (A), D11.1 (A), D12.1 (A), D7.1 (A), D8.1 (A), D9.1 (A); no longer D10.2 (K), D11.2 (K), D12.2 (K), D7.2 (K), D8.2 (K), D9.2 (K)
- net at R7.2: now also D10.2 (K); no longer D10.1 (A)
- net at R10.2: now also D7.2 (K); no longer D7.1 (A)
- net at R8.2: now also D11.2 (K); no longer D11.1 (A)
- net at R11.2: now also D8.2 (K); no longer D8.1 (A)
- net at R9.2: now also D12.2 (K); no longer D12.1 (A)
- net at R12.2: now also D9.2 (K); no longer D9.1 (A)
Changed lines of the file:
@@
 EESchema Schematic File Version 2
+LIBS:FilPilote-rescue
 LIBS:power
 LIBS:device
@@
 LIBS:memory
 LIBS:xilinx
-LIBS:special
 LIBS:microcontrollers
 LIBS:dsp
@@
 LIBS:w_connectors
 LIBS:FilPilote-cache
-EELAYER 24 0
+EELAYER 25 0
 EELAYER END
 $Descr A4 11693 8268
@@
 $EndDescr
 $Comp
-L MOC3041M IC1
+L MOC3041M-RESCUE-FilPilote IC1
 U 1 1 55FE75A9
 P 1800 1450
@@
 $EndComp
 $Comp
-L MOC3041M IC2
+L MOC3041M-RESCUE-FilPilote IC2
 U 1 1 55FE7673
 P 1800 1950
@@
 $EndComp
 $Comp
-L R R1
+L R-RESCUE-FilPilote R1
 U 1 1 55FE76CA
 P 2400 1350
@@
 $EndComp
 $Comp
-L R R2
+L R-RESCUE-FilPilote R2
 U 1 1 55FE7725
 P 2400 1850
@@
 $EndComp
 $Comp
-L R R7
+L R-RESCUE-FilPilote R7
 U 1 1 55FE7750
 P 2650 2100
@@
 $EndComp
 $Comp
-L R R10
+L R-RESCUE-FilPilote R10
 U 1 1 55FE77A8
 P 2800 2250
@@
 	1    0    0    -1
 $EndComp
-$Comp
-L LED D10
-U 1 1 55FE77DF
-P 2400 2350
-F 0 "D10" H 2400 2450 50  0000 C CNN
-F 1 "LED" H 2400 2250 50  0000 C CNN
-F 2 "LEDs:LED-3MM" H 2400 2350 60  0001 C CNN
-F 3 "" H 2400 2350 60  0000 C CNN
-	1    2400 2350
-	-1   0    0    1
-$EndComp
-$Comp
-L LED D7
-U 1 1 55FE7858
-P 2100 2500
-F 0 "D7" H 2100 2600 50  0000 C CNN
-F 1 "LED" H 2100 2400 50  0000 C CNN
-F 2 "LEDs:LED-3MM" H 2100 2500 60  0001 C CNN
-F 3 "" H 2100 2500 60  0000 C CNN
-	1    2100 2500
-	-1   0    0    1
-$EndComp
 Wire Wire Line
 	2650 1350 3050 1350
@@
 	2650 1850 3050 1850
 $Comp
-L GND #PWR1
+L GND-RESCUE-FilPilote #PWR01
 U 1 1 55FE7984
 P 1700 2500
-F 0 "#PWR1" H 1700 2500 30  0001 C CNN
+F 0 "#PWR01" H 1700 2500 30  0001 C CNN
 F 1 "GND" H 1700 2430 30  0001 C CNN
 F 2 "" H 1700 2500 60  0000 C CNN
@@
 F 0 "D1" H 1250 1650 40  0000 C CNN
 F 1 "1N4007" H 1250 1450 40  0000 C CNN
-F 2 "Diodes_ThroughHole:Diode_DO-41_SOD81_Horizontal_RM10" H 1250 1550 60  0001 C CNN
+F 2 "Discret:D4" H 1250 1550 60  0001 C CNN
 F 3 "" H 1250 1550 60  0000 C CNN
 	1    1250 1550
@@
 F 0 "D2" H 1250 2150 40  0000 C CNN
 F 1 "1N4007" H 1250 1950 40  0000 C CNN
-F 2 "Diodes_ThroughHole:Diode_DO-41_SOD81_Horizontal_RM10" H 1250 2050 60  0001 C CNN
+F 2 "Discret:D4" H 1250 2050 60  0001 C CNN
 F 3 "" H 1250 2050 60  0000 C CNN
 	1    1250 2050
@@
 	2800 1350 2800 2000
 $Comp
-L MOC3041M IC3
+L MOC3041M-RESCUE-FilPilote IC3
 U 1 1 55FE8888
 P 1800 3100
@@
 $EndComp
 $Comp
-L MOC3041M IC4
+L MOC3041M-RESCUE-FilPilote IC4
 U 1 1 55FE888E
 P 1800 3600
@@
 $EndComp
 $Comp
-L R R3
+L R-RESCUE-FilPilote R3
 U 1 1 55FE8894
 P 2400 3000
@@
 $EndComp
 $Comp
-L R R4
+L R-RESCUE-FilPilote R4
 U 1 1 55FE889A
 P 2400 3500
@@
 $EndComp
 $Comp
-L R R8
+L R-RESCUE-FilPilote R8
 U 1 1 55FE88A0
 P 2650 3750
@@
 $EndComp
 $Comp
-L R R11
+L R-RESCUE-FilPilote R11
 U 1 1 55FE88A6
 P 2800 3900
@@
 	1    0    0    -1
 $EndComp
-$Comp
-L LED D11
-U 1 1 55FE88AC
-P 2400 4000
-F 0 "D11" H 2400 4100 50  0000 C CNN
-F 1 "LED" H 2400 3900 50  0000 C CNN
-F 2 "LEDs:LED-3MM" H 2400 4000 60  0001 C CNN
-F 3 "" H 2400 4000 60  0000 C CNN
-	1    2400 4000
-	-1   0    0    1
-$EndComp
-$Comp
-L LED D8
-U 1 1 55FE88B2
-P 2100 4150
-F 0 "D8" H 2100 4250 50  0000 C CNN
-F 1 "LED" H 2100 4050 50  0000 C CNN
-F 2 "LEDs:LED-3MM" H 2100 4150 60  0001 C CNN
-F 3 "" H 2100 4150 60  0000 C CNN
-	1    2100 4150
-	-1   0    0    1
-$EndComp
 Wire Wire Line
 	2650 3000 3050 3000
@@
 	2650 3500 3050 3500
 $Comp
-L GND #PWR2
+L GND-RESCUE-FilPilote #PWR02
 U 1 1 55FE88BB
 P 1700 4150
-F 0 "#PWR2" H 1700 4150 30  0001 C CNN
+F 0 "#PWR02" H 1700 4150 30  0001 C CNN
 F 1 "GND" H 1700 4080 30  0001 C CNN
 F 2 "" H 1700 4150 60  0000 C CNN
@@
 F 0 "D3" H 1250 3300 40  0000 C CNN
 F 1 "1N4007" H 1250 3100 40  0000 C CNN
-F 2 "Diodes_ThroughHole:Diode_DO-41_SOD81_Horizontal_RM10" H 1250 3200 60  0001 C CNN
+F 2 "Discret:D4" H 1250 3200 60  0001 C CNN
 F 3 "" H 1250 3200 60  0000 C CNN
 	1    1250 3200
@@
 F 0 "D4" H 1250 3800 40  0000 C CNN
 F 1 "1N4007" H 1250 3600 40  0000 C CNN
-F 2 "Diodes_ThroughHole:Diode_DO-41_SOD81_Horizontal_RM10" H 1250 3700 60  0001 C CNN
+F 2 "Discret:D4" H 1250 3700 60  0001 C CNN
 F 3 "" H 1250 3700 60  0000 C CNN
 	1    1250 3700
@@
 	2800 3000 2800 3650
 $Comp
-L MOC3041M IC5
+L MOC3041M-RESCUE-FilPilote IC5
 U 1 1 55FE9478
 P 1800 4750
@@
 $EndComp
 $Comp
-L MOC3041M IC6
+L MOC3041M-RESCUE-FilPilote IC6
 U 1 1 55FE947E
 P 1800 5250
@@
 $EndComp
 $Comp
-L R R5
+L R-RESCUE-FilPilote R5
 U 1 1 55FE9484
 P 2400 4650
@@
 $EndComp
 $Comp
-L R R6
+L R-RESCUE-FilPilote R6
 U 1 1 55FE948A
 P 2400 5150
@@
 $EndComp
 $Comp
-L R R9
+L R-RESCUE-FilPilote R9
 U 1 1 55FE9490
 P 2650 5400
@@
 $EndComp
 $Comp
-L R R12
+L R-RESCUE-FilPilote R12
 U 1 1 55FE9496
 P 2800 5550
@@
 	1    0    0    -1
 $EndComp
-$Comp
-L LED D12
-U 1 1 55FE949C
-P 2400 5650
-F 0 "D12" H 2400 5750 50  0000 C CNN
-F 1 "LED" H 2400 5550 50  0000 C CNN
-F 2 "LEDs:LED-3MM" H 2400 5650 60  0001 C CNN
-F 3 "" H 2400 5650 60  0000 C CNN
-	1    2400 5650
-	-1   0    0    1
-$EndComp
-$Comp
-L LED D9
-U 1 1 55FE94A2
-P 2100 5800
-F 0 "D9" H 2100 5900 50  0000 C CNN
-F 1 "LED" H 2100 5700 50  0000 C CNN
-F 2 "LEDs:LED-3MM" H 2100 5800 60  0001 C CNN
-F 3 "" H 2100 5800 60  0000 C CNN
-	1    2100 5800
-	-1   0    0    1
-$EndComp
 Wire Wire Line
 	2650 4650 3050 4650
@@
 	2650 5150 3050 5150
 $Comp
-L GND #PWR3
+L GND-RESCUE-FilPilote #PWR03
 U 1 1 55FE94AB
 P 1700 5800
-F 0 "#PWR3" H 1700 5800 30  0001 C CNN
+F 0 "#PWR03" H 1700 5800 30  0001 C CNN
 F 1 "GND" H 1700 5730 30  0001 C CNN
 F 2 "" H 1700 5800 60  0000 C CNN
@@
 F 0 "D5" H 1250 4950 40  0000 C CNN
 F 1 "1N4007" H 1250 4750 40  0000 C CNN
-F 2 "Diodes_ThroughHole:Diode_DO-41_SOD81_Horizontal_RM10" H 1250 4850 60  0001 C CNN
+F 2 "Discret:D4" H 1250 4850 60  0001 C CNN
 F 3 "" H 1250 4850 60  0000 C CNN
 	1    1250 4850
@@
 F 0 "D6" H 1250 5450 40  0000 C CNN
 F 1 "1N4007" H 1250 5250 40  0000 C CNN
-F 2 "Diodes_ThroughHole:Diode_DO-41_SOD81_Horizontal_RM10" H 1250 5350 60  0001 C CNN
+F 2 "Discret:D4" H 1250 5350 60  0001 C CNN
 F 3 "" H 1250 5350 60  0000 C CNN
 	1    1250 5350
@@
 Cmd-3
 $Comp
-L GND #PWR4
+L GND-RESCUE-FilPilote #PWR04
 U 1 1 55FF87EA
 P 7250 6350
-F 0 "#PWR4" H 7250 6350 30  0001 C CNN
+F 0 "#PWR04" H 7250 6350 30  0001 C CNN
 F 1 "GND" H 7250 6280 30  0001 C CNN
 F 2 "" H 7250 6350 60  0000 C CNN
@@
 $EndComp
 $Comp
-L PWR_FLAG #FLG1
+L PWR_FLAG #FLG05
 U 1 1 55FF882F
 P 7250 6350
-F 0 "#FLG1" H 7250 6445 30  0001 C CNN
+F 0 "#FLG05" H 7250 6445 30  0001 C CNN
 F 1 "PWR_FLAG" H 7250 6530 30  0000 C CNN
 F 2 "" H 7250 6350 60  0000 C CNN
@@
 	9350 1800 9500 1800
 $Comp
-L GND #PWR5
+L GND-RESCUE-FilPilote #PWR06
 U 1 1 55FFB8E1
 P 9500 2100
-F 0 "#PWR5" H 9500 2100 30  0001 C CNN
+F 0 "#PWR06" H 9500 2100 30  0001 C CNN
 F 1 "GND" H 9500 2030 30  0001 C CNN
 F 2 "" H 9500 2100 60  0000 C CNN
@@
 	5150 1300 5150 1200
 NoConn ~ 5150 1100
+$Comp
+L LED D10
+U 1 1 5607FB2B
+P 2400 2350
+F 0 "D10" H 2400 2450 50  0000 C CNN
+F 1 "LED" H 2400 2250 50  0000 C CNN
+F 2 "LEDs:LED-3MM" H 2400 2350 60  0001 C CNN
+F 3 "" H 2400 2350 60  0000 C CNN
+	1    2400 2350
+	1    0    0    -1
+$EndComp
+$Comp
+L LED D7
+U 1 1 5607FBD5
+P 2100 2500
+F 0 "D7" H 2100 2600 50  0000 C CNN
+F 1 "LED" H 2100 2400 50  0000 C CNN
+F 2 "LEDs:LED-3MM" H 2100 2500 60  0001 C CNN
+F 3 "" H 2100 2500 60  0000 C CNN
+	1    2100 2500
+	1    0    0    -1
+$EndComp
+$Comp
+L LED D8
+U 1 1 56080C97
+P 2100 4150
+F 0 "D8" H 2100 4250 50  0000 C CNN
+F 1 "LED" H 2100 4050 50  0000 C CNN
+F 2 "LEDs:LED-3MM" H 2100 4150 60  0001 C CNN
+F 3 "" H 2100 4150 60  0000 C CNN
+	1    2100 4150
+	1    0    0    -1
+$EndComp
+$Comp
+L LED D11
+U 1 1 56080D41
+P 2400 4000
+F 0 "D11" H 2400 4100 50  0000 C CNN
+F 1 "LED" H 2400 3900 50  0000 C CNN
+F 2 "LEDs:LED-3MM" H 2400 4000 60  0001 C CNN
+F 3 "" H 2400 4000 60  0000 C CNN
+	1    2400 4000
+	1    0    0    -1
+$EndComp
+$Comp
+L LED D9
+U 1 1 560814F5
+P 2100 5800
+F 0 "D9" H 2100 5900 50  0000 C CNN
+F 1 "LED" H 2100 5700 50  0000 C CNN
+F 2 "LEDs:LED-3MM" H 2100 5800 60  0001 C CNN
+F 3 "" H 2100 5800 60  0000 C CNN
+	1    2100 5800
+	1    0    0    -1
+$EndComp
+$Comp
+L LED D12
+U 1 1 560815A3
+P 2400 5650
+F 0 "D12" H 2400 5750 50  0000 C CNN
+F 1 "LED" H 2400 5550 50  0000 C CNN
+F 2 "LEDs:LED-3MM" H 2400 5650 60  0001 C CNN
+F 3 "" H 2400 5650 60  0000 C CNN
+	1    2400 5650
+	1    0    0    -1
+$EndComp
 $EndSCHEMATC
